Commit message: 20180423_2

File: catkin_ur/src/universal_robot-kinetic-devel/ur_description/urdf/ur5withdouble.urdf.xacro (robot description, xacro)
@@ -10,5 +10,5 @@
   <parent link="world" />
   <child link = "head_plate_frame" />
-  <origin xyz="0.0 0.0 0.0" rpy="0.0 0.0 0.0" />
+  <origin xyz="0.0 0.0 0.0" rpy="0.0 0.0 1.57" />
 </joint>
 <link name="head_plate_frame">
